File: STMF401.kicad_sch (KiCad schematic)
At the start: 16 parts, among them J6 Conn_01x04_Pin, Y1 X322525MQB4SI

Commit message: feat: added mani lines for GND
Parts:
- added C26, C33: 0.1u, Capacitor_SMD:C_0805_2012Metric_Pad1.18x1.45mm_HandSolder, symbol Device:C_Small
Connections:
- net +3V3D: no longer C15.1, C16.1
- net +3V3_MCU: now also C15.1, C16.1, C26.1, C33.1
- net GND: now also C26.2, C33.2
- no-connect marks 0 -> 17
Other:
- moved on the sheet: C14, C15, C16, L1
