File: External_interfaces.kicad_sch (KiCad schematic)
At the start: 26 parts, among them J10 Conn_01x06_Pin, J15 Conn_01x02_Pin, J7 Conn_01x02_Pin, J8 Conn_01x06_Pin, J9 Conn_01x02_Pin, Q1 AO3400A, Q2 AO3400A

Commit message: feat: добавлены все элементы схемы, начал соединение сигнгальных линий к микроконтроллеру
Parts:
- added C52: 0.1u, Capacitor_SMD:C_0805_2012Metric_Pad1.18x1.45mm_HandSolder, symbol Device:C_Small
- added J17: Conn_01x04_Pin, Connector_PinSocket_2.54mm:PinSocket_1x04_P2.54mm_Vertical, symbol Connector:Conn_01x04_Pin
- added R31, R32: 0, Resistor_SMD:R_0805_2012Metric_Pad1.20x1.40mm_HandSolder, symbol Device:R
- added VD15: GSOT03C-E3-08, Package_TO_SOT_SMD:SOT-23_Handsoldering, symbol TWS:GSOT03C-E3-08
Connections:
- net +3V3D: now also R31.1
- net +5V: now also R32.1
- net GND: now also C52.2, J17.1 (Pin_1), VD15.3 (A)
- net DEBUG_RX renamed DEBUG_RX1
- net DEBUG_TX renamed DEBUG_TX1
- new net: C52.1, J17.4 (Pin_4), R31.2, R32.2
- new net DEBUG_RX2: J17.2 (Pin_2), VD15.1 (K1)
- new net DEBUG_TX2: J17.3 (Pin_3), VD15.2 (K2)

Commit message: feat: Разведены линии питания
Parts:
- VD10, VD15, VD2, VD3: footprint Package_TO_SOT_SMD:SOT-23_Handsoldering -> Package_TO_SOT_SMD:SOT-23
Changed lines of the file:
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@@
 			)
 		)
-		(property "Footprint" "Package_TO_SOT_SMD:SOT-23_Handsoldering"
+		(property "Footprint" "Package_TO_SOT_SMD:SOT-23"
 			(at 143.51 59.69 0)
 			(hide yes)
@@
 			)
 		)
-		(property "Footprint" "Package_TO_SOT_SMD:SOT-23_Handsoldering"
+		(property "Footprint" "Package_TO_SOT_SMD:SOT-23"
 			(at 76.2 172.72 0)
 			(hide yes)
@@
 			)
 		)
-		(property "Footprint" "Package_TO_SOT_SMD:SOT-23_Handsoldering"
+		(property "Footprint" "Package_TO_SOT_SMD:SOT-23"
 			(at 67.31 59.69 0)
 			(hide yes)
@@
 			)
 		)
-		(property "Footprint" "Package_TO_SOT_SMD:SOT-23_Handsoldering"
+		(property "Footprint" "Package_TO_SOT_SMD:SOT-23"
 			(at 64.77 116.84 0)
 			(hide yes)
