File: PWR.kicad_sch (KiCad schematic)
At the start: 32 parts, among them J1 Conn_01x02_Pin, U2 XC6206P332MR, U4 MCP6001-OT, U5 AMS1117-3.3, U6 XL1509-5.0

Commit message: feat: добавлены все элементы схемы, начал соединение сигнгальных линий к микроконтроллеру
Parts:
- U6: footprint Package_SO:SOIC-8_3.9x4.9mm_P1.27mm -> Package_SO:SOIC-8-1EP_3.9x4.9mm_P1.27mm_EP2.29x3mm_ThermalVias
Changed lines of the file:
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@@
 			)
 		)
-		(property "Footprint" "Package_SO:SOIC-8_3.9x4.9mm_P1.27mm"
+		(property "Footprint" "Package_SO:SOIC-8-1EP_3.9x4.9mm_P1.27mm_EP2.29x3mm_ThermalVias"
 			(at 88.9 102.108 0)
 			(hide yes)

Commit message: feat: добавлены светодиоды, размещены почти все компоненты кроме модулей IMU
Parts:
- VD4: footprint Package_TO_SOT_SMD:SOT-23_Handsoldering -> Package_TO_SOT_SMD:SOT-23
Changed lines of the file:
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@@
 			)
 		)
-		(property "Footprint" "Package_TO_SOT_SMD:SOT-23_Handsoldering"
+		(property "Footprint" "Package_TO_SOT_SMD:SOT-23"
 			(at 176.53 76.2 0)
 			(hide yes)

Commit message: feat: Разведены линии питания
Parts:
- U2: footprint Package_TO_SOT_SMD:SOT-23_Handsoldering -> Package_TO_SOT_SMD:SOT-23
Changed lines of the file:
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@@
 			)
 		)
-		(property "Footprint" "Package_TO_SOT_SMD:SOT-23_Handsoldering"
+		(property "Footprint" "Package_TO_SOT_SMD:SOT-23"
 			(at 236.22 105.156 0)
 			(hide yes)
